File: kamstrup-wifi.brd (EAGLE design)
At the start: 36 x 89.3 mm, 21 parts, among them T1 BT137, T2 BT137, U1 ESP8266-07

Commit message: Version sent to pcb fabrication
Parts:
- moved FOCA 4.00 mm to (16.7, 26.9)
Other:
- board text added: "v.1.4.3"
- board text removed: "v.1.4.2"
Changed lines of the file:
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@@
 <hole x="1.5" y="14" drill="2.2"/>
 <hole x="21.5" y="38.6" drill="2.2"/>
-<text x="21.74875" y="32.45625" size="1.016" layer="25" rot="R90" align="center-left">VCC</text>
-<text x="19.20875" y="32.45625" size="1.016" layer="25" rot="R90" align="center-left">TxD</text>
-<text x="16.66875" y="32.45625" size="1.016" layer="25" rot="R90" align="center-left">RxD</text>
+<text x="21.74875" y="28.45625" size="1.016" layer="25" rot="R90" align="center-left">VCC</text>
+<text x="19.20875" y="28.45625" size="1.016" layer="25" rot="R90" align="center-left">TxD</text>
+<text x="16.66875" y="28.45625" size="1.016" layer="25" rot="R90" align="center-left">RxD</text>
 <text x="7.46125" y="18.89125" size="1.016" layer="25" ratio="10" rot="R270">ESP8266
 ESP-07</text>
-<text x="7.46125" y="29.68625" size="1.016" layer="25" ratio="15" rot="R270">v.1.4.2</text>
-<text x="26.82875" y="32.45625" size="1.016" layer="25" rot="R90" align="center-left">GND</text>
+<text x="7.46125" y="29.68625" size="1.016" layer="25" ratio="15" rot="R270">v.1.4.3</text>
+<text x="26.82875" y="28.45625" size="1.016" layer="25" rot="R90" align="center-left">GND</text>
 <text x="20.7725" y="75.615" size="1.27" layer="25" ratio="20" rot="R90" align="center">AC IN
 N   L</text>
-<text x="27.6225" y="13.0175" size="1.016" layer="26" font="fixed" rot="MR0">Part            RS#
+<text x="26.6225" y="10.0175" size="1.016" layer="26" font="fixed" rot="MR0">Part            RS#
 JP1, JP2, JP3   821-8701
 KAM             702-2937
@@
 T1, T2          792-0709
 </text>
-<wire x1="28.41625" y1="26.845" x2="14.7875" y2="26.845" width="0.1524" layer="26"/>
-<wire x1="14.7875" y1="26.845" x2="5.08" y2="26.845" width="0.1524" layer="26"/>
-<wire x1="5.08" y1="26.845" x2="5.08" y2="13.81125" width="0.1524" layer="26"/>
-<wire x1="5.08" y1="13.81125" x2="14.7875" y2="13.81125" width="0.1524" layer="26"/>
-<wire x1="14.7875" y1="13.81125" x2="28.41625" y2="13.81125" width="0.1524" layer="26"/>
-<wire x1="28.41625" y1="13.81125" x2="28.41625" y2="26.845" width="0.1524" layer="26"/>
-<wire x1="14.7875" y1="26.845" x2="14.7875" y2="13.81125" width="0.1524" layer="26"/>
+<wire x1="27.41625" y1="23.845" x2="13.7875" y2="23.845" width="0.1524" layer="26"/>
+<wire x1="13.7875" y1="23.845" x2="4.08" y2="23.845" width="0.1524" layer="26"/>
+<wire x1="4.08" y1="23.845" x2="4.08" y2="10.81125" width="0.1524" layer="26"/>
+<wire x1="4.08" y1="10.81125" x2="13.7875" y2="10.81125" width="0.1524" layer="26"/>
+<wire x1="13.7875" y1="10.81125" x2="27.41625" y2="10.81125" width="0.1524" layer="26"/>
+<wire x1="27.41625" y1="10.81125" x2="27.41625" y2="23.845" width="0.1524" layer="26"/>
+<wire x1="13.7875" y1="23.845" x2="13.7875" y2="10.81125" width="0.1524" layer="26"/>
 <wire x1="12.99375" y1="80.06" x2="16.9625" y2="80.06" width="0.254" layer="25"/>
 <wire x1="16.9625" y1="80.06" x2="16.9625" y2="70.2175" width="0.254" layer="25"/>
@@
 <attribute name="VALUE" x="0.19" y="31.825" size="1.27" layer="27"/>
 </element>
-<element name="FOCA" library="SparkFun-Connectors" package="1X05" value="" x="16.66875" y="30.86125" smashed="yes">
-<attribute name="NAME" x="14.20495" y="28.56255" size="1.27" layer="25" ratio="10" rot="R90"/>
-<attribute name="VALUE" x="15.39875" y="27.68625" size="1.27" layer="27"/>
+<element name="FOCA" library="SparkFun-Connectors" package="1X05" value="" x="16.66875" y="26.86125" smashed="yes">
+<attribute name="NAME" x="14.20495" y="24.56255" size="1.27" layer="25" ratio="10" rot="R90"/>
+<attribute name="VALUE" x="15.39875" y="23.68625" size="1.27" layer="27"/>
 </element>
 <element name="PRG" library="SparkFun-Connectors" package="1X02" value="M02PTH" x="5.87375" y="8.5725" smashed="yes" rot="R180">
@@
 <wire x1="25.7175" y1="1.74625" x2="23.8125" y2="1.74625" width="0.4064" layer="16"/>
 <wire x1="23.8125" y1="1.74625" x2="16.66875" y2="8.89" width="0.4064" layer="16"/>
-<wire x1="16.66875" y1="8.89" x2="16.66875" y2="30.86125" width="0.4064" layer="16"/>
+<wire x1="16.66875" y1="8.89" x2="16.66875" y2="26.86125" width="0.4064" layer="16"/>
 <wire x1="6.54" y1="37.54" x2="11.99" y2="37.54" width="0.4064" layer="16"/>
 <wire x1="11.99" y1="37.54" x2="16.66875" y2="32.86125" width="0.4064" layer="16"/>
-<wire x1="16.66875" y1="32.86125" x2="16.66875" y2="30.86125" width="0.4064" layer="16"/>
+<wire x1="16.66875" y1="32.86125" x2="16.66875" y2="26.86125" width="0.4064" layer="16"/>
 </signal>
 <signal name="N$2">
@@
 <wire x1="25.4" y1="4.6875" x2="25.4" y2="3.65125" width="0.4064" layer="1"/>
 <wire x1="25.4" y1="3.65125" x2="24.765" y2="3.01625" width="0.4064" layer="1"/>
-<wire x1="19.20875" y1="30.86125" x2="19.20875" y2="8.5725" width="0.4064" layer="16"/>
+<wire x1="19.20875" y1="26.86125" x2="19.20875" y2="8.5725" width="0.4064" layer="16"/>
 <wire x1="19.20875" y1="8.5725" x2="24.765" y2="3.01625" width="0.4064" layer="16"/>
 <wire x1="5.23875" y1="39.52875" x2="12.54125" y2="39.52875" width="0.4064" layer="16"/>
 <wire x1="12.54125" y1="39.52875" x2="19.20875" y2="32.86125" width="0.4064" layer="16"/>
-<wire x1="19.20875" y1="32.86125" x2="19.20875" y2="30.86125" width="0.4064" layer="16"/>
+<wire x1="19.20875" y1="32.86125" x2="19.20875" y2="26.86125" width="0.4064" layer="16"/>
 </signal>
 <signal name="N$4">
@@
 <wire x1="19.3675" y1="20.745" x2="19.4125" y2="20.7" width="0.4064" layer="1"/>
 <contactref element="R8" pad="1"/>
-<wire x1="19.3675" y1="20.745" x2="19.3675" y2="27.5275" width="0.4064" layer="1"/>
-<wire x1="19.3675" y1="27.5275" x2="20.6375" y2="28.7975" width="0.4064" layer="1"/>
-<wire x1="20.6375" y1="28.7975" x2="28.09875" y2="28.7975" width="0.4064" layer="1"/>
-<wire x1="28.09875" y1="28.7975" x2="29.36875" y2="30.0675" width="0.4064" layer="1"/>
-<wire x1="29.36875" y1="30.0675" x2="29.36875" y2="34.76875" width="0.4064" layer="1"/>
+<wire x1="19.3675" y1="20.745" x2="19.3675" y2="23.0275" width="0.4064" layer="1"/>
+<wire x1="19.3675" y1="23.0275" x2="20.6375" y2="24.2975" width="0.4064" layer="1"/>
+<wire x1="20.6375" y1="24.2975" x2="28.09875" y2="24.2975" width="0.4064" layer="1"/>
+<wire x1="28.09875" y1="24.2975" x2="29.36875" y2="25.5675" width="0.4064" layer="1"/>
+<wire x1="29.36875" y1="25.5675" x2="29.36875" y2="34.76875" width="0.4064" layer="1"/>
 <wire x1="29.36875" y1="34.76875" x2="27.14625" y2="36.99125" width="0.4064" layer="1"/>
 </signal>
